Commit message: Gazebo Configuring

File: description/robot_core.xacro (robot description, xacro)
@@ -31,4 +31,7 @@
         </xacro:inertial_box>
     </link>
+    <gazebo reference="chassis">
+            <material>Gazebo/White </material>
+    </gazebo>
     <!-- LEFT WHEEL -->
         <joint name="left_wheel_joint" type="continuous">
@@ -54,6 +57,9 @@
             </xacro:inertial_cylinder>
         </link>
+        <gazebo reference="left_wheel">
+            <material>Gazebo/Blue </material>
+        </gazebo>
     <!-- RIGHT WHEEL-->
-    <joint name="right_wheel_joint" type="continuous">
+        <joint name="right_wheel_joint" type="continuous">
             <parent link="base_link"/>
             <child link="right_wheel"/>
@@ -77,4 +83,7 @@
             </xacro:inertial_cylinder>
         </link>
+        <gazebo reference="right_wheel">
+            <material>Gazebo/Blue </material>
+        </gazebo>
     <!-- CASTER WHEEL LINK -->
     <joint name="caster_wheel_joint" type="fixed">
@@ -99,3 +108,8 @@
         </xacro:inertial_sphere>
     </link>
+    <gazebo reference="caster_wheel">
+        <material>Gazebo/Black</material>
+        <mu1 value="0.001"/>
+        <mu2 value="0.001"/>
+    </gazebo>
 </robot>
